Commit message: fix the initial pose of the arm

File: smart_arm_description/urdf/smart_arm_description.urdf.xacro (robot description, xacro)
@@ -758,5 +758,5 @@
       velocity="1" />
   </joint>
-  <joint name="wrist_lower_joint" type="revolute">
+  <joint name="wrist_middle_joint" type="revolute">
     <origin
       xyz="0 -0.063543 0.017875"
@@ -765,5 +765,5 @@
       link="wrist_link" />
     <child
-      link="wrist_lower_link" />
+      link="wrist_middle_link" />
     <axis
       xyz="-1 0 0" />
@@ -772,55 +772,7 @@
       upper="1"
       effort="5"
-      velocity="5" />
-  </joint>
-  <joint name="pinky_1_joint" type="revolute">
-    <origin
-      xyz="-0.043751 0.0091577 0.05009"
-      rpy="-1.6708 -0.61679 0.12536" />
-    <parent
-      link="wrist_lower_link" />
-    <child
-      link="pinky_1_link" />
-    <axis
-      xyz="-1 0 0" />
-    <limit
-      lower="-1"
-      upper="1"
-      effort="5"
       velocity="2" />
   </joint>
-  <joint name="pinky_2_joint" type="revolute">
-    <origin
-      xyz="-0.00023197 -0.029503 0.0045349"
-      rpy="3.026 0.13765 -0.015931" />
-    <parent
-      link="pinky_1_link" />
-    <child
-      link="pinky_2_link" />
-    <axis
-      xyz="-0.99042 0 0.13812" />
-    <limit
-      lower="-1"
-      upper="1"
-      effort="5"
-      velocity="3" />
-  </joint>
-  <joint name="pinky_3_joint" type="revolute">
-    <origin
-      xyz="-0.0011308 0.018906 -0.0033205"
-      rpy="-0.24361 0.13856 0" />
-    <parent
-      link="pinky_2_link" />
-    <child
-      link="pinky_3_link" />
-    <axis
-      xyz="-1 0 0" />
-    <limit
-      lower="-1"
-      upper="1"
-      effort="5"
-      velocity="2" />
-  </joint>
-  <joint name="wrist_middle_joint" type="revolute">
+  <joint name="wrist_lower_joint" type="revolute">
     <origin
       xyz="0 -0.063543 0.017875"
@@ -829,7 +781,71 @@
       link="wrist_link" />
     <child
+      link="wrist_lower_link" />
+    <axis
+      xyz="-1 0 0" />
+    <limit
+      lower="-1"
+      upper="1"
+      effort="5"
+      velocity="5" />
+  </joint>
+  <joint name="pinky_1_joint" type="revolute">
+    <origin
+      xyz="-0.043751 0.0091577 0.05009"
+      rpy="-1.5908 -0.61679 0.12536" />
+    <parent
+      link="wrist_lower_link" />
+    <child
+      link="pinky_1_link" />
+    <axis
+      xyz="1 0 0" />
+    <limit
+      lower="-1"
+      upper="1"
+      effort="5"
+      velocity="2" />
+  </joint>
+  <joint name="pinky_2_joint" type="revolute">
+    <origin
+      xyz="-0.00023197 -0.029503 0.0045349"
+      rpy="3.226 0.13765 -0.015931" />
+    <parent
+      link="pinky_1_link" />
+    <child
+      link="pinky_2_link" />
+    <axis
+      xyz="1 0 0" />
+    <limit
+      lower="-1"
+      upper="1"
+      effort="5"
+      velocity="3" />
+  </joint>
+  <joint name="pinky_3_joint" type="revolute">
+    <origin
+      xyz="-0.0011308 0.018906 -0.0033205"
+      rpy="0.24361 0.13856 0" />
+    <parent
+      link="pinky_2_link" />
+    <child
+      link="pinky_3_link" />
+    <axis
+      xyz="1 0 0" />
+    <limit
+      lower="-1"
+      upper="1"
+      effort="5"
+      velocity="2" />
+  </joint>
+  <joint name="ring_1_joint" type="revolute">
+    <origin
+      xyz="-0.069801 0.0076347 0.041426"
+      rpy="1.5238 -0.78078 0.17561" />
+    <parent
       link="wrist_middle_link" />
-    <axis
-      xyz="-1 0 0" />
+    <child
+      link="ring_1_link" />
+    <axis
+      xyz="1 0 0" />
     <limit
       lower="-1"
@@ -838,14 +854,14 @@
       velocity="2" />
   </joint>
-  <joint name="ring_1_joint" type="revolute">
-    <origin
-      xyz="-0.069801 0.0076347 0.041426"
-      rpy="1.3238 -0.78078 0.17561" />
-    <parent
-      link="wrist_middle_link" />
-    <child
+  <joint name="ring_2_joint" type="revolute">
+    <origin
+      xyz="-0.00027831 0.035204 -0.0065715"
+      rpy="-0.08653 0 0" />
+    <parent
       link="ring_1_link" />
-    <axis
-      xyz="-1 0 0" />
+    <child
+      link="ring_2_link" />
+    <axis
+      xyz="1 0 0" />
     <limit
       lower="-1"
@@ -854,30 +870,14 @@
       velocity="2" />
   </joint>
-  <joint name="ring_2_joint" type="revolute">
-    <origin
-      xyz="-0.00027831 0.035204 -0.0065715"
-      rpy="-0.14653 0 0" />
-    <parent
-      link="ring_1_link" />
-    <child
+  <joint name="ring_3_joint" type="revolute">
+    <origin
+      xyz="-0.000793430469754296 0.0229811955997807 -0.00184137348495991"
+      rpy="-0.183278724594159 0 0" />
+    <parent
       link="ring_2_link" />
-    <axis
-      xyz="-1 0 0" />
-    <limit
-      lower="-1"
-      upper="1"
-      effort="5"
-      velocity="2" />
-  </joint>
-  <joint name="ring_3_joint" type="revolute">
-    <origin
-      xyz="-0.000793430469754296 0.0229811955997807 -0.00184137348495991"
-      rpy="-0.143278724594159 0 0" />
-    <parent
-      link="ring_2_link" />
     <child
       link="ring_3_link" />
     <axis
-      xyz="-1 0 0" />
+      xyz="1 0 0" />
     <limit
       lower="-1"
@@ -905,5 +905,5 @@
     <origin
       xyz="-0.041192 0.017697 -0.032051"
-      rpy="-0.75622 0.31508 0.77256" />
+      rpy="-1 0.31508 0.77256" />
     <parent
       link="wrist_upper_link" />
@@ -911,5 +911,5 @@
       link="thumb_1_link" />
     <axis
-      xyz="-1 0 0" />
+      xyz="1 0 0" />
     <limit
       lower="-1"
@@ -921,5 +921,5 @@
     <origin
       xyz="-0.000865682899112985 0.0214109109835155 0.0182563649065549"
-      rpy="0.640757193595075 0 0" />
+      rpy="0 0 0" />
     <parent
       link="thumb_1_link" />
@@ -927,5 +927,5 @@
       link="thumb_2_link" />
     <axis
-      xyz="-1 0 0" />
+      xyz="1 0 0" />
     <limit
       lower="-1"
@@ -937,5 +937,5 @@
     <origin
       xyz="0.000525788242336553 -0.0208949853387586 0.107469880482186"
-      rpy="1.5707963267949 0 -1.5707963267949" />
+      rpy="1.8507963267949 0 -1.5707963267949" />
     <parent
       link="wrist_link" />
@@ -943,5 +943,5 @@
       link="middle_1_link" />
     <axis
-      xyz="-0.999716298839136 -0.0238185187486232 0" />
+      xyz="1 0 0" />
     <limit
       lower="-1"
@@ -953,5 +953,5 @@
     <origin
       xyz="-0.0011154 0.03449 -0.015386"
-      rpy="-0.3814 0 0.023821" />
+      rpy="-0.2614 0 0.023821" />
     <parent
       link="middle_1_link" />
@@ -959,5 +959,5 @@
       link="middle_2_link" />
     <axis
-      xyz="-1 0 0" />
+      xyz="1 0 0" />
     <limit
       lower="-1"
@@ -969,5 +969,5 @@
     <origin
       xyz="-0.00083707 0.024267 -0.0016433"
-      rpy="-0.13093 0 0" />
+      rpy="0.45093 0 0" />
     <parent
       link="middle_2_link" />
@@ -975,5 +975,5 @@
       link="middle_3_link" />
     <axis
-      xyz="-1 0 0" />
+      xyz="1 0 0" />
     <limit
       lower="-1"
@@ -991,5 +991,5 @@
       link="pointer_1_link" />
     <axis
-      xyz="-1 0 0" />
+      xyz="1 0 0" />
     <limit
       lower="-1"
@@ -1001,5 +1001,5 @@
     <origin
       xyz="-0.00027831 0.03552 -0.0045641"
-      rpy="-0.089775 0 0" />
+      rpy="0.840000 0 0" />
     <parent
       link="pointer_1_link" />
@@ -1007,5 +1007,5 @@
       link="pointer_2_link" />
     <axis
-      xyz="-1 0 0" />
+      xyz="1 0 0" />
     <limit
       lower="-1"
@@ -1017,5 +1017,5 @@
     <origin
       xyz="-0.00079343 0.014451 -0.017972"
-      rpy="-0.95742 0 0" />
+      rpy="-0.91742 0 0" />
     <parent
       link="pointer_2_link" />
@@ -1023,5 +1023,5 @@
       link="pointer_3_link" />
     <axis
-      xyz="-1 0 0" />
+      xyz="1 0 0" />
     <limit
       lower="-1"

Commit message: rearranaged jointsin urdf

File: smart_arm_description/urdf/smart_arm_description.urdf.xacro (robot description, xacro)
@@ -758,4 +758,20 @@
       velocity="1" />
   </joint>
+  <joint name="wrist_upper_joint" type="revolute">
+    <origin
+      xyz="0 0.00467160843217863 0.00716947951775644"
+      rpy="0 1.48772480012052 -1.5707963267949" />
+    <parent
+      link="wrist_link" />
+    <child
+      link="wrist_upper_link" />
+    <axis
+      xyz="-1 0 0" />
+    <limit
+      lower="-1"
+      upper="1"
+      effort="5"
+      velocity="3" />
+  </joint>
   <joint name="wrist_middle_joint" type="revolute">
     <origin
@@ -790,4 +806,36 @@
       velocity="5" />
   </joint>
+  <joint name="thumb_1_joint" type="revolute">
+    <origin
+      xyz="-0.041192 0.017697 -0.032051"
+      rpy="-1 0.31508 0.77256" />
+    <parent
+      link="wrist_upper_link" />
+    <child
+      link="thumb_1_link" />
+    <axis
+      xyz="1 0 0" />
+    <limit
+      lower="-1"
+      upper="1"
+      effort="5"
+      velocity="4" />
+  </joint>
+  <joint name="thumb_2_joint" type="revolute">
+    <origin
+      xyz="-0.000865682899112985 0.0214109109835155 0.0182563649065549"
+      rpy="0 0 0" />
+    <parent
+      link="thumb_1_link" />
+    <child
+      link="thumb_2_link" />
+    <axis
+      xyz="1 0 0" />
+    <limit
+      lower="-1"
+      upper="1"
+      effort="5"
+      velocity="4" />
+  </joint>
   <joint name="pinky_1_joint" type="revolute">
     <origin
@@ -886,52 +934,4 @@
       velocity="2" />
   </joint>
-  <joint name="wrist_upper_joint" type="revolute">
-    <origin
-      xyz="0 0.00467160843217863 0.00716947951775644"
-      rpy="0 1.48772480012052 -1.5707963267949" />
-    <parent
-      link="wrist_link" />
-    <child
-      link="wrist_upper_link" />
-    <axis
-      xyz="-1 0 0" />
-    <limit
-      lower="-1"
-      upper="1"
-      effort="5"
-      velocity="3" />
-  </joint>
-  <joint name="thumb_1_joint" type="revolute">
-    <origin
-      xyz="-0.041192 0.017697 -0.032051"
-      rpy="-1 0.31508 0.77256" />
-    <parent
-      link="wrist_upper_link" />
-    <child
-      link="thumb_1_link" />
-    <axis
-      xyz="1 0 0" />
-    <limit
-      lower="-1"
-      upper="1"
-      effort="5"
-      velocity="4" />
-  </joint>
-  <joint name="thumb_2_joint" type="revolute">
-    <origin
-      xyz="-0.000865682899112985 0.0214109109835155 0.0182563649065549"
-      rpy="0 0 0" />
-    <parent
-      link="thumb_1_link" />
-    <child
-      link="thumb_2_link" />
-    <axis
-      xyz="1 0 0" />
-    <limit
-      lower="-1"
-      upper="1"
-      effort="5"
-      velocity="4" />
-  </joint>
   <joint name="middle_1_joint" type="revolute">
     <origin

Commit message: metacarpals joint limits according to anatomical ranges

File: smart_arm_description/urdf/smart_arm_description.urdf.xacro (robot description, xacro)
@@ -742,4 +742,8 @@
     </collision>
   </link>
+  <xacro:property name="very_small_limit" value="-0.1"/>
+  <xacro:property name="proximal_finger_joint_limit" value="1.5707"/>
+  <xacro:property name="middle_finger_joint_limit" value="1.3707"/>
+  <xacro:property name="distal_finger_joint_limit" value="1.2707"/>
   <joint name="wrist_joint" type="revolute">
     <origin
@@ -817,6 +821,6 @@
       xyz="1 0 0" />
     <limit
-      lower="-1"
-      upper="1"
+      lower="${very_small_limit}"
+      upper="0.8720"
       effort="5"
       velocity="4" />
@@ -833,6 +837,6 @@
       xyz="1 0 0" />
     <limit
-      lower="-1"
-      upper="1"
+      lower="${very_small_limit}"
+      upper="1.39626"
       effort="5"
       velocity="4" />
@@ -847,8 +851,8 @@
       link="pinky_1_link" />
     <axis
-      xyz="1 0 0" />
-    <limit
-      lower="-1"
-      upper="1"
+      xyz="-1 0 0" />
+    <limit
+      lower="${very_small_limit}"
+      upper="${proximal_finger_joint_limit}"
       effort="5"
       velocity="2" />
@@ -863,8 +867,8 @@
       link="pinky_2_link" />
     <axis
-      xyz="1 0 0" />
-    <limit
-      lower="-1"
-      upper="1"
+      xyz="-1 0 0" />
+    <limit
+      lower="${very_small_limit}"
+      upper="${middle_finger_joint_limit}"
       effort="5"
       velocity="3" />
@@ -879,8 +883,8 @@
       link="pinky_3_link" />
     <axis
-      xyz="1 0 0" />
-    <limit
-      lower="-1"
-      upper="1"
+      xyz="-1 0 0" />
+    <limit
+      lower="${very_small_limit}"
+      upper="${distal_finger_joint_limit}"
       effort="5"
       velocity="2" />
@@ -895,8 +899,8 @@
       link="ring_1_link" />
     <axis
-      xyz="1 0 0" />
-    <limit
-      lower="-1"
-      upper="1"
+      xyz="-1 0 0" />
+    <limit
+      lower="${very_small_limit}"
+      upper="${proximal_finger_joint_limit}"
       effort="5"
       velocity="2" />
@@ -911,8 +915,8 @@
       link="ring_2_link" />
     <axis
-      xyz="1 0 0" />
-    <limit
-      lower="-1"
-      upper="1"
+      xyz="-1 0 0" />
+    <limit
+      lower="${very_small_limit}"
+      upper="${middle_finger_joint_limit}"
       effort="5"
       velocity="2" />
@@ -927,8 +931,8 @@
       link="ring_3_link" />
     <axis
-      xyz="1 0 0" />
-    <limit
-      lower="-1"
-      upper="1"
+      xyz="-1 0 0" />
+    <limit
+      lower="${very_small_limit}"
+      upper="${distal_finger_joint_limit}"
       effort="5"
       velocity="2" />
@@ -943,8 +947,8 @@
       link="middle_1_link" />
     <axis
-      xyz="1 0 0" />
-    <limit
-      lower="-1"
-      upper="1"
+      xyz="-1 0 0" />
+    <limit
+      lower="${very_small_limit}"
+      upper="${proximal_finger_joint_limit}"
       effort="5"
       velocity="5" />
@@ -959,8 +963,8 @@
       link="middle_2_link" />
     <axis
-      xyz="1 0 0" />
-    <limit
-      lower="-1"
-      upper="1"
+      xyz="-1 0 0" />
+    <limit
+      lower="${very_small_limit}"
+      upper="${middle_finger_joint_limit}"
       effort="5"
       velocity="4" />
@@ -975,8 +979,8 @@
       link="middle_3_link" />
     <axis
-      xyz="1 0 0" />
-    <limit
-      lower="-1"
-      upper="1"
+      xyz="-1 0 0" />
+    <limit
+      lower="${very_small_limit}"
+      upper="${distal_finger_joint_limit}"
       effort="4"
       velocity="5" />
@@ -991,8 +995,8 @@
       link="pointer_1_link" />
     <axis
-      xyz="1 0 0" />
-    <limit
-      lower="-1"
-      upper="1"
+      xyz="-1 0 0" />
+    <limit
+      lower="${very_small_limit}"
+      upper="${proximal_finger_joint_limit}"
       effort="5"
       velocity="2" />
@@ -1007,8 +1011,8 @@
       link="pointer_2_link" />
     <axis
-      xyz="1 0 0" />
-    <limit
-      lower="-1"
-      upper="1"
+      xyz="-1 0 0" />
+    <limit
+      lower="${very_small_limit}"
+      upper="${middle_finger_joint_limit}"
       effort="5"
       velocity="3" />
@@ -1023,8 +1027,8 @@
       link="pointer_3_link" />
     <axis
-      xyz="1 0 0" />
-    <limit
-      lower="-1"
-      upper="1"
+      xyz="-1 0 0" />
+    <limit
+      lower="${very_small_limit}"
+      upper="${distal_finger_joint_limit}"
       effort="5"
       velocity="2" />

Commit message: fix wrist joints limits

File: smart_arm_description/urdf/smart_arm_description.urdf.xacro (robot description, xacro)
@@ -755,8 +755,8 @@
       link="wrist_link" />
     <axis
-      xyz="0 -1 0" />
-    <limit
-      lower="-1"
-      upper="1"
+      xyz="0 1 0" />
+    <limit
+      lower="-0.872665"
+      upper="0.872665"
       effort="5"
       velocity="1" />
@@ -771,8 +771,8 @@
       link="wrist_upper_link" />
     <axis
-      xyz="-1 0 0" />
-    <limit
-      lower="-1"
-      upper="1"
+      xyz="1 0 0" />
+    <limit
+      lower="${very_small_limit}"
+      upper="0.872665"
       effort="5"
       velocity="3" />
@@ -789,6 +789,6 @@
       xyz="-1 0 0" />
     <limit
-      lower="-1"
-      upper="1"
+      lower="${very_small_limit}"
+      upper="${-very_small_limit}"
       effort="5"
       velocity="2" />
@@ -805,6 +805,6 @@
       xyz="-1 0 0" />
     <limit
-      lower="-1"
-      upper="1"
+      lower="${very_small_limit}"
+      upper="${-very_small_limit}"
       effort="5"
       velocity="5" />
